File: SNES/JACR_SNES.kicad_sch (KiCad schematic)
At the start: 4 parts, among them J1 JACR CARTRIDGE ADAPTER, J2 SNES Cartridge Slot

Commit message: JACR connector was modified, voltage pins were changed
Connections:
- net +5V: now also J1.79 (+5V), J1.80 (+5V); no longer J1.75 (+5V)
- no-connect marks 22 -> 21
Changed lines of the file:
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@@
 	)
 	(no_connect
-		(at 59.69 132.08)
+		(at 34.29 43.18)
 	)
 	(no_connect
-		(at 34.29 132.08)
+		(at 59.69 132.08)
 	)
 	(no_connect
-		(at 59.69 142.24)
+		(at 34.29 132.08)
 	)
 	(no_connect
@@
 	)
 	(no_connect
-		(at 34.29 43.18)
+		(at 59.69 43.18)
 	)
 	(no_connect
@@
 	)
 	(no_connect
+		(at 34.29 137.16)
+	)
+	(no_connect
 		(at 106.68 132.08)
 	)
@@
 	)
 	(no_connect
-		(at 34.29 142.24)
-	)
-	(no_connect
 		(at 59.69 134.62)
 	)
 	(no_connect
-		(at 59.69 43.18)
-	)
-	(no_connect
 		(at 59.69 48.26)
 	)
@@
 	)
 	(symbol
-		(lib_id "power:+5V")
-		(at 34.29 137.16 90)
-		(unit 1)
-		(exclude_from_sim no)
-		(in_bom yes)
-		(on_board yes)
-		(dnp no)
-		(fields_autoplaced yes)
-		(property "Reference" "#PWR08"
-			(at 38.1 137.16 0)
-			(effects
-				(font
-					(size 1.27 1.27)
-				)
-				(hide yes)
-			)
-		)
-		(property "Value" "+5V"
-			(at 30.48 137.1599 90)
-			(effects
-				(font
-					(size 1.27 1.27)
-				)
-				(justify left)
-			)
-		)
-		(property "Footprint" ""
-			(at 34.29 137.16 0)
-			(effects
-				(font
-					(size 1.27 1.27)
-				)
-				(hide yes)
-			)
-		)
-		(property "Datasheet" ""
-			(at 34.29 137.16 0)
-			(effects
-				(font
-					(size 1.27 1.27)
-				)
-				(hide yes)
-			)
-		)
-		(property "Description" "Power symbol creates a global label with name \"+5V\""
-			(at 34.29 137.16 0)
-			(effects
-				(font
-					(size 1.27 1.27)
-				)
-				(hide yes)
-			)
-		)
-		(pin "1"
-		)
-		(instances
-			(project ""
-				(path "/b312f5ab-7935-4830-b125-a7ec355c500e"
-					(reference "#PWR08")
-					(unit 1)
-				)
-			)
-		)
-	)
-	(symbol
 		(lib_id "Nintendo:SNES_Cartridge_Slot")
 		(at 127 91.44 0)
@@
 	)
 	(symbol
+		(lib_id "power:+5V")
+		(at 59.69 142.24 270)
+		(mirror x)
+		(unit 1)
+		(exclude_from_sim no)
+		(in_bom yes)
+		(on_board yes)
+		(dnp no)
+		(property "Reference" "#PWR013"
+			(at 55.88 142.24 0)
+			(effects
+				(font
+					(size 1.27 1.27)
+				)
+				(hide yes)
+			)
+		)
+		(property "Value" "+5V"
+			(at 63.5 142.2399 90)
+			(effects
+				(font
+					(size 1.27 1.27)
+				)
+				(justify left)
+			)
+		)
+		(property "Footprint" ""
+			(at 59.69 142.24 0)
+			(effects
+				(font
+					(size 1.27 1.27)
+				)
+				(hide yes)
+			)
+		)
+		(property "Datasheet" ""
+			(at 59.69 142.24 0)
+			(effects
+				(font
+					(size 1.27 1.27)
+				)
+				(hide yes)
+			)
+		)
+		(property "Description" "Power symbol creates a global label with name \"+5V\""
+			(at 59.69 142.24 0)
+			(effects
+				(font
+					(size 1.27 1.27)
+				)
+				(hide yes)
+			)
+		)
+		(pin "1"
+		)
+		(instances
+			(project "JACR_SNES"
+				(path "/b312f5ab-7935-4830-b125-a7ec355c500e"
+					(reference "#PWR013")
+					(unit 1)
+				)
+			)
+		)
+	)
+	(symbol
 		(lib_id "power:GND")
 		(at 193.04 78.74 0)
@@
 					(unit 1)
 				)
+			)
+		)
+	)
+	(symbol
+		(lib_id "power:+5V")
+		(at 34.29 142.24 90)
+		(unit 1)
+		(exclude_from_sim no)
+		(in_bom yes)
+		(on_board yes)
+		(dnp no)
+		(fields_autoplaced yes)
+		(property "Reference" "#PWR08"
+			(at 38.1 142.24 0)
+			(effects
+				(font
+					(size 1.27 1.27)
+				)
+				(hide yes)
+			)
+		)
+		(property "Value" "+5V"
+			(at 30.48 142.2399 90)
+			(effects
+				(font
+					(size 1.27 1.27)
+				)
+				(justify left)
+			)
+		)
+		(property "Footprint" ""
+			(at 34.29 142.24 0)
+			(effects
+				(font
+					(size 1.27 1.27)
+				)
+				(hide yes)
+			)
+		)
+		(property "Datasheet" ""
+			(at 34.29 142.24 0)
+			(effects
+				(font
+					(size 1.27 1.27)
+				)
+				(hide yes)
+			)
+		)
+		(property "Description" "Power symbol creates a global label with name \"+5V\""
+			(at 34.29 142.24 0)
+			(effects
+				(font
+					(size 1.27 1.27)
+				)
+				(hide yes)
+			)
+		)
+		(pin "1"
+		)
+		(instances
+			(project ""
+				(path "/b312f5ab-7935-4830-b125-a7ec355c500e"
+					(reference "#PWR08")
+					(unit 1)
+				)
